Commit message: Add other dogs. Add simple pd controller.

File: legged_robots/legged_robots_sims/urdf/hyq/common.xacro (robot description, xacro)
@@ -1,4 +1,4 @@
 <?xml version="1.0"?>
-<robot xmlns:xacro="http://ros.org/wiki/xacro">
+<robot xmlns:xacro="http://www.ros.org/wiki/xacro">
 	<xacro:property name="PI" value="3.1415926535897931"/>
     <!-- kin limits (sign ref is RH leg)-->

File: legged_robots/legged_robots_sims/urdf/hyq/hyq.urdf.xacro (robot description, xacro)
@@ -1,5 +1,6 @@
 <?xml version="1.0"?>
-<robot name="hyq" xmlns:xacro="http://ros.org/wiki/xacro">
-<!-- The following included files set up definitions of parts of the robot body -->
+<robot name="hyq" xmlns:xacro="http://www.ros.org/wiki/xacro">
+  <xacro:include filename="$(find legged_robots_sims)/urdf/hyq/hyq.gazebo.xacro" />
+  <!-- The following included files set up definitions of parts of the robot body -->
   <xacro:include filename="$(find legged_robots_sims)/urdf/hyq/common.xacro"/>
 	<!-- HyQ trunk -->

File: legged_robots/legged_robots_sims/urdf/hyq/leg.urdf.xacro (robot description, xacro)
@@ -1,4 +1,4 @@
 <?xml version="1.0"?>
-<robot xmlns:xacro="http://ros.org/wiki/xacro">
+<robot xmlns:xacro="http://www.ros.org/wiki/xacro">
 	<!-- leg macro definiction -->
 	<xacro:macro name="hyq_leg" params="name parent *origin reflect_hip reflect_upper reflect_front">
@@ -37,4 +37,34 @@
 			<child  link="${name}_foot"/>
 		</joint>
+		<transmission name="${name}_haa_joint_trans">
+      		<type>transmission_interface/SimpleTransmission</type>
+      		<joint name="${name}_haa_joint">
+        		<hardwareInterface>hardware_interface/EffortJointInterface</hardwareInterface>
+      		</joint>
+      		<actuator name="${name}_haa_joint_motor">
+        		<hardwareInterface>hardware_interface/EffortJointInterface</hardwareInterface>
+        		<mechanicalReduction>1</mechanicalReduction>
+      		</actuator>
+    	</transmission>
+		<transmission name="${name}_hfe_joint_trans">
+      		<type>transmission_interface/SimpleTransmission</type>
+      		<joint name="${name}_hfe_joint">
+        		<hardwareInterface>hardware_interface/EffortJointInterface</hardwareInterface>
+      		</joint>
+      		<actuator name="${name}_hfe_joint_motor">
+        		<hardwareInterface>hardware_interface/EffortJointInterface</hardwareInterface>
+        		<mechanicalReduction>1</mechanicalReduction>
+      		</actuator>
+    	</transmission>
+		<transmission name="${name}_kfe_joint_trans">
+      		<type>transmission_interface/SimpleTransmission</type>
+      		<joint name="${name}_kfe_joint">
+        		<hardwareInterface>hardware_interface/EffortJointInterface</hardwareInterface>
+      		</joint>
+      		<actuator name="${name}_kfe_joint_motor">
+        		<hardwareInterface>hardware_interface/EffortJointInterface</hardwareInterface>
+        		<mechanicalReduction>1</mechanicalReduction>
+      		</actuator>
+    	</transmission>
 		<!-- Links -->
 		<!-- Hip assembly link -->

File: legged_robots/legged_robots_sims/urdf/hyq/trunk.urdf.xacro (robot description, xacro)
@@ -1,4 +1,4 @@
 <?xml version="1.0"?>
-<robot xmlns:xacro="http://ros.org/wiki/xacro">
+<robot xmlns:xacro="http://www.ros.org/wiki/xacro">
 	<!-- trunk macro definition -->
 	<xacro:macro name="hyq_trunk" params="name">
