Commit message: Addition urdf and lauch file of  hyq_fixed model

File: legged_robots/legged_robots_sims/urdf/hyq_fixed/trunk.urdf.xacro (robot description, xacro)
@@ -3,9 +3,11 @@
 	<!-- trunk macro definition -->
 	<xacro:macro name="hyq_trunk" params="name">
-		<!-- Floating-base Joint -->
-		<joint name="floating_base" type="fixed">
-			<origin xyz="0 0 0.0" rpy="0 0 0"/>
-			<parent link="${name}"/>
-			<child link="trunk"/>
+		<!-- World -->
+		<link name="world"/>
+		<!-- World Fixed Joint-->
+  		<joint name="world_base_joint" type="fixed">
+    		<origin xyz="0 0 ${z_offset_from_world}" rpy="0 0 0" />
+			<parent link="world" />
+			<child link="${name}" />
 		</joint>
 		<!-- Footprint link -->
@@ -17,4 +19,10 @@
 			</visual>
 		</link>
+		<!-- Floating-base Joint -->
+		<joint name="floating_base" type="fixed">
+			<origin xyz="0 0 0.0" rpy="0 0 0"/>
+			<parent link="${name}"/>
+			<child link="trunk"/>
+		</joint>
 		<!-- Trunk link -->
 		<link name="trunk">
