Commit message: Add Leg Forward Kinematics

File: legged_robots/legged_robots_sims/urdf/hyq_fixed/hyq.urdf.xacro (robot description, xacro)
@@ -1,7 +1,7 @@
 <?xml version="1.0"?>
 <robot name="hyq" xmlns:xacro="http://www.ros.org/wiki/xacro">
-  <xacro:include filename="$(find legged_robots_sims)/urdf/hyq_fixed/hyq.gazebo.xacro" />
-  <!-- The following included files set up definitions of parts of the robot body -->
-  <xacro:include filename="$(find legged_robots_sims)/urdf/hyq_fixed/common.xacro"/>
+    <xacro:include filename="$(find legged_robots_sims)/urdf/hyq_fixed/hyq.gazebo.xacro" />
+    <!-- The following included files set up definitions of parts of the robot body -->
+    <xacro:include filename="$(find legged_robots_sims)/urdf/hyq_fixed/common.xacro"/>
 	<!-- HyQ trunk -->
 	<xacro:include filename="$(find legged_robots_sims)/urdf/hyq_fixed/trunk.urdf.xacro"/>

File: legged_robots/legged_robots_sims/urdf/hyq_fixed/leg.urdf.xacro (robot description, xacro)
@@ -11,4 +11,5 @@
 			<axis xyz="0 0 1"/>
 			<limit effort="${haa_limit}" velocity="12.0" lower="${haa_min*PI/180}" upper="${haa_max*PI/180}" />
+			<dynamics damping="100" friction="1000" />
 		</joint>
 		<!-- Upper leg joint -->
@@ -19,6 +20,7 @@
 			<axis xyz="0 0 1"/>
 			<limit effort="150.0" velocity="12.0"
-          lower="${-(1+reflect_front)*5*PI/36-(1-reflect_front)*7*PI/36}"
-          upper="${(1-reflect_front)*5*PI/36+(1+reflect_front)*7*PI/36}"/>
+          		   lower="${-(1+reflect_front)*5*PI/36-(1-reflect_front)*7*PI/36}"
+          		   upper="${(1-reflect_front)*5*PI/36+(1+reflect_front)*7*PI/36}"/>
+		    <dynamics damping="100" friction="1000" />
 		</joint>
 		<!-- Lower leg joint -->
@@ -29,6 +31,7 @@
 			<axis xyz="0 0 1"/>
 			<limit effort="150.0" velocity="12.0"
-          lower="${-(1+reflect_front)*7*PI/18+(1-reflect_front)*PI/18}"
-          upper="${(1-reflect_front)*7*PI/18-(1+reflect_front)*PI/18}"/>
+          		   lower="${-(1+reflect_front)*7*PI/18+(1-reflect_front)*PI/18}"
+                   upper="${(1-reflect_front)*7*PI/18-(1+reflect_front)*PI/18}"/>
+		    <dynamics damping="100" friction="1000" />
 		</joint>
 		<!-- Foot joint -->
