Commit message: Split leg_controller into header and cpp. Add service to update gain.

File: legged_robots/legged_robots_description/urdf/hyq_fixed/leg.urdf.xacro (robot description, xacro)
@@ -11,4 +11,5 @@
 			<axis xyz="0 0 1"/>
 			<limit effort="${haa_limit}" velocity="12.0" lower="${haa_min*PI/180}" upper="${haa_max*PI/180}" />
+			<dynamics damping="0" friction="1000000000" />
 		</joint>
 		<!-- Upper leg joint -->
@@ -21,4 +22,5 @@
           lower="${-(1+reflect_front)*5*PI/36-(1-reflect_front)*7*PI/36}"
           upper="${(1-reflect_front)*5*PI/36+(1+reflect_front)*7*PI/36}"/>
+		  	<dynamics damping="0" friction="1000000000" />
 		</joint>
 		<!-- Lower leg joint -->
@@ -31,4 +33,5 @@
           lower="${-(1+reflect_front)*7*PI/18+(1-reflect_front)*PI/18}"
           upper="${(1-reflect_front)*7*PI/18-(1+reflect_front)*PI/18}"/>
+		  	<!-- <dynamics damping="100000" friction="100000" /> -->
 		</joint>
 		<!-- Foot joint -->
