Commit message: Add forward kinematics/inverse dynamics of each legs and virtual spring damper controller

File: legged_robots/legged_robots_description/urdf/hyq/leg.urdf.xacro (robot description, xacro)
@@ -10,5 +10,8 @@
 			<child  link="${name}_hipassembly"/>
 			<axis xyz="0 0 1"/>
-			<limit effort="${haa_limit}" velocity="12.0" lower="${haa_min*PI/180}" upper="${haa_max*PI/180}" />
+			<limit effort="${haa_limit}" velocity="12.0"
+			lower="-${2*PI}" upper="${2*PI}"/>
+			<!-- lower="${haa_min*PI/180}" upper="${haa_max*PI/180}" />		 -->
+			<dynamics damping="0" friction="0" />
 		</joint>
 		<!-- Upper leg joint -->
@@ -19,6 +22,8 @@
 			<axis xyz="0 0 1"/>
 			<limit effort="150.0" velocity="12.0"
-          lower="${-(1+reflect_front)*5*PI/36-(1-reflect_front)*7*PI/36}"
-          upper="${(1-reflect_front)*5*PI/36+(1+reflect_front)*7*PI/36}"/>
+          lower="-${2*PI}" upper="${2*PI}"/>
+          <!-- lower="${-(1+reflect_front)*5*PI/36-(1-reflect_front)*7*PI/36}"
+          upper="${(1-reflect_front)*5*PI/36+(1+reflect_front)*7*PI/36}"/> -->
+		  	<dynamics damping="0" friction="0" />
 		</joint>
 		<!-- Lower leg joint -->
@@ -29,6 +34,8 @@
 			<axis xyz="0 0 1"/>
 			<limit effort="150.0" velocity="12.0"
-          lower="${-(1+reflect_front)*7*PI/18+(1-reflect_front)*PI/18}"
-          upper="${(1-reflect_front)*7*PI/18-(1+reflect_front)*PI/18}"/>
+          lower="-${2*PI}" upper="${2*PI}"/>
+          <!-- lower="${-(1+reflect_front)*7*PI/18+(1-reflect_front)*PI/18}"
+          upper="${(1-reflect_front)*7*PI/18-(1+reflect_front)*PI/18}"/> -->
+		  	<dynamics damping="0" friction="0" />
 		</joint>
 		<!-- Foot joint -->

File: legged_robots/legged_robots_description/urdf/hyq/trunk.urdf.xacro (robot description, xacro)
@@ -5,5 +5,5 @@
 		<!-- Floating-base Joint -->
 		<joint name="floating_base" type="fixed">
-			<origin xyz="0 0 0.0" rpy="0 0 0"/>
+			<origin xyz="0 0 1" rpy="0 0 0"/>
 			<parent link="${name}"/>
 			<child link="trunk"/>

File: legged_robots/legged_robots_description/urdf/hyq_fixed/leg.urdf.xacro (robot description, xacro)
@@ -10,6 +10,8 @@
 			<child  link="${name}_hipassembly"/>
 			<axis xyz="0 0 1"/>
-			<limit effort="${haa_limit}" velocity="12.0" lower="${haa_min*PI/180}" upper="${haa_max*PI/180}" />
-			<dynamics damping="0" friction="1000000000" />
+			<limit effort="${haa_limit}" velocity="12.0"
+			lower="-${2*PI}" upper="${2*PI}"/>
+			<!-- lower="${haa_min*PI/180}" upper="${haa_max*PI/180}" />		 -->
+			<!-- <dynamics damping="0" friction="10000" /> -->
 		</joint>
 		<!-- Upper leg joint -->
@@ -20,7 +22,8 @@
 			<axis xyz="0 0 1"/>
 			<limit effort="150.0" velocity="12.0"
-          lower="${-(1+reflect_front)*5*PI/36-(1-reflect_front)*7*PI/36}"
-          upper="${(1-reflect_front)*5*PI/36+(1+reflect_front)*7*PI/36}"/>
-		  	<dynamics damping="0" friction="1000000000" />
+			lower="-${2*PI}" upper="${2*PI}"/>
+          <!-- lower="${-(1+reflect_front)*5*PI/36-(1-reflect_front)*7*PI/36}"
+          upper="${(1-reflect_front)*5*PI/36+(1+reflect_front)*7*PI/36}"/> -->
+		  	<!-- <dynamics damping="0" friction="10000" /> -->
 		</joint>
 		<!-- Lower leg joint -->
@@ -34,5 +37,5 @@
           <!-- lower="${-(1+reflect_front)*7*PI/18+(1-reflect_front)*PI/18}"
           upper="${(1-reflect_front)*7*PI/18-(1+reflect_front)*PI/18}"/> -->
-		  	<!-- <dynamics damping="100000" friction="100000" /> -->
+		  	<!-- <dynamics damping="0" friction="10000" /> -->
 		</joint>
 		<!-- Foot joint -->

Commit message: Add stand alone.

File: legged_robots/legged_robots_description/urdf/hyq/leg.urdf.xacro (robot description, xacro)
@@ -155,4 +155,6 @@
 				<material name="black" />
 			</visual>
+			<gazebo>
+			</gazebo>
 		</link>
 	</xacro:macro>

File: legged_robots/legged_robots_description/urdf/hyq/trunk.urdf.xacro (robot description, xacro)
@@ -5,5 +5,5 @@
 		<!-- Floating-base Joint -->
 		<!-- <joint name="floating_base" type="fixed">
-			<origin xyz="0 0 1" rpy="0 0 0"/>
+			<origin xyz="0 0 0.5" rpy="0 0 0"/>
 			<parent link="${name}"/>
 			<child link="trunk"/>
@@ -16,5 +16,5 @@
 				</geometry>
 			</visual>
-		</link> --> -->
+		</link> -->
 		<!-- Trunk link -->
 		<link name="trunk">
