Commit message: Subscribe gazebo link states. Not finished.

File: legged_robots/legged_robots_description/urdf/hyq/trunk.urdf.xacro (robot description, xacro)
@@ -4,11 +4,11 @@
 	<xacro:macro name="hyq_trunk" params="name">
 		<!-- Floating-base Joint -->
-		<joint name="floating_base" type="fixed">
+		<!-- <joint name="floating_base" type="fixed">
 			<origin xyz="0 0 1" rpy="0 0 0"/>
 			<parent link="${name}"/>
 			<child link="trunk"/>
-		</joint>
+		</joint> -->
 		<!-- Footprint link -->
-		<link name="${name}">
+		<!-- <link name="${name}">
 			<visual>
 				<geometry>
@@ -16,5 +16,5 @@
 				</geometry>
 			</visual>
-		</link>
+		</link> --> -->
 		<!-- Trunk link -->
 		<link name="trunk">

Commit message: Fix foot slip.

File: legged_robots/legged_robots_description/urdf/hyq/trunk.urdf.xacro (robot description, xacro)
@@ -5,5 +5,5 @@
 		<!-- Floating-base Joint -->
 		<!-- <joint name="floating_base" type="fixed">
-			<origin xyz="0 0 0.5" rpy="0 0 0"/>
+			<origin xyz="0 0 1" rpy="0 0 0"/>
 			<parent link="${name}"/>
 			<child link="trunk"/>
