Commit message: Modify balance controller. it's working, but need more tuning.

File: legged_robots/legged_robots_description/urdf/hyq/common.xacro (robot description, xacro)
@@ -36,4 +36,5 @@
 	<xacro:property name="zcom_hipassembly" value="0.16931"/>
 	<xacro:property name="m_hipassembly" value="2.93"/>
+	<!-- <xacro:property name="m_hipassembly" value="0.1"/> -->
 	<xacro:property name="ixx_hipassembly" value="0.05071"/>
 	<xacro:property name="iyy_hipassembly" value="0.05486"/>
@@ -47,4 +48,5 @@
 	<xacro:property name="zcom_upperleg" value="0.0"/>
 	<xacro:property name="m_upperleg" value="2.638"/>
+	<!-- <xacro:property name="m_upperleg" value="0.1"/> -->
 	<xacro:property name="ixx_upperleg" value="0.00368"/>
 	<xacro:property name="iyy_upperleg" value="0.02719"/>
@@ -58,4 +60,5 @@
 	<xacro:property name="zcom_lowerleg" value="-0.0001"/>
 	<xacro:property name="m_lowerleg" value="0.881"/>
+	<!-- <xacro:property name="m_lowerleg" value="0.1"/> -->
 	<xacro:property name="ixx_lowerleg" value="0.00047"/>
 	<xacro:property name="iyy_lowerleg" value="0.01256"/>
