Commit message: imu apply test

File: legged_robots/legged_robots_description/urdf/hyq/hyq.urdf.xacro (robot description, xacro)
@@ -8,4 +8,6 @@
 	<!-- HyQ legs -->
 	<xacro:include filename="$(find legged_robots_description)/urdf/hyq/leg.urdf.xacro"/>
+    <!-- HyQ sensors -->
+	<xacro:include filename="$(find sensors_description)/urdfs/sensors/microstrain_3dmgx425_imu.urdf.xacro"/>
 	<!-- Using the macros defined above -->
 	<!-- trunk -->
@@ -47,3 +49,11 @@
 		<origin xyz="${-d_fh/2} ${-d_lr/2} 0" rpy="0 ${PI/2} 0"/>
 	</xacro:hyq_leg>
+	<!-- IMU trunk -->
+	<xacro:microstrain_3dmgx425_imu
+		parent="trunk"
+		imu_name="trunk_imu"
+		imu_topic="trunk_imu_1/data"
+		update_rate="250">
+		<origin xyz="0.290 0.000 0.0999214" rpy="0 ${-PI} 0"/>
+	</xacro:microstrain_3dmgx425_imu>
 </robot>

Commit message: Contact sensor test
using hyq_description

File: legged_robots/legged_robots_description/urdf/hyq/hyq.urdf.xacro (robot description, xacro)
@@ -1,4 +1,5 @@
 <?xml version="1.0"?>
 <robot name="hyq" xmlns:xacro="http://www.ros.org/wiki/xacro">
+<xacro:arg name="load_force_sensors" default="true"/>
   <xacro:include filename="$(find legged_robots_description)/urdf/hyq/hyq.gazebo.xacro" />
   <!-- The following included files set up definitions of parts of the robot body -->
@@ -19,5 +20,6 @@
 		reflect_hip="1"
 		reflect_upper="1"
-		reflect_front="1">
+		reflect_front="1"
+		load_force_sensors="$(arg load_force_sensors)">
 		<origin xyz="${d_fh/2} ${d_lr/2} 0" rpy="0 ${PI/2} ${PI}"/>
 	</xacro:hyq_leg>
@@ -28,5 +30,6 @@
 		reflect_hip="-1"
 		reflect_upper="-1"
-		reflect_front="1">
+		reflect_front="1"
+		load_force_sensors="$(arg load_force_sensors)">
 		<origin xyz="${d_fh/2} ${-d_lr/2} 0" rpy="0 ${PI/2} 0"/>
 	</xacro:hyq_leg>
@@ -37,5 +40,6 @@
 		reflect_hip="-1"
 		reflect_upper="1"
-		reflect_front="-1">
+		reflect_front="-1"
+		load_force_sensors="$(arg load_force_sensors)">
 		<origin xyz="${-d_fh/2} ${d_lr/2} 0" rpy="0 ${PI/2} ${PI}"/>
 	</xacro:hyq_leg>
@@ -46,5 +50,6 @@
 		reflect_hip="1"
 		reflect_upper="-1"
-		reflect_front="-1">
+		reflect_front="-1"
+		load_force_sensors="$(arg load_force_sensors)">
 		<origin xyz="${-d_fh/2} ${-d_lr/2} 0" rpy="0 ${PI/2} 0"/>
 	</xacro:hyq_leg>

File: legged_robots/legged_robots_description/urdf/hyq/leg.urdf.xacro (robot description, xacro)
@@ -1,6 +1,7 @@
 <?xml version="1.0"?>
 <robot xmlns:xacro="http://www.ros.org/wiki/xacro">
+	<xacro:include filename="$(find legged_robots_description)/urdf/hyq/leg.gazebo.xacro"/>
 	<!-- leg macro definiction -->
-	<xacro:macro name="hyq_leg" params="name parent *origin reflect_hip reflect_upper reflect_front">
+	<xacro:macro name="hyq_leg" params="name parent *origin reflect_hip reflect_upper reflect_front load_force_sensors">
 		<!-- Joints -->
 		<!-- Hip assembly joint -->
@@ -158,4 +159,5 @@
 			</gazebo>
 		</link>
+		<xacro:leg_gazebo name="${name}" load_force_sensors="${load_force_sensors}"/>
 	</xacro:macro>
 </robot>

File: legged_robots/legged_robots_description/urdf/hyq/trunk.urdf.xacro (robot description, xacro)
@@ -1,4 +1,5 @@
 <?xml version="1.0"?>
 <robot xmlns:xacro="http://www.ros.org/wiki/xacro">
+<xacro:include filename="$(find legged_robots_description)/urdf/hyq/trunk.gazebo.xacro"/>
 	<!-- trunk macro definition -->
 	<xacro:macro name="hyq_trunk" params="name">
